File: Hertz200/PCB_DESIGN/HERTZ200/BQ24195_SMPS.kicad_sch (KiCad schematic)
At the start: 35 parts, among them J4 Jack-DC, J5 USB_B_Mini, Q3 Si2312DS, Q4 CSD25302Q2, Q5 Si2312DS, U5 BQ24195LRGER

Commit message: schamtics_finish
Parts:
- gave numbers to parts that had none: 5
Changed lines of the file:
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@@
     (stroke (width 0) (type default) (color 0 0 0 0))
+  )
+  (polyline (pts (xy 92.71 134.62) (xy 198.12 134.62))
+    (stroke (width 1) (type default) (color 0 0 0 0))
   )
   (wire (pts (xy 240.03 83.82) (xy 240.03 86.36))
@@
   )
   (wire (pts (xy 48.26 97.79) (xy 48.26 99.06))
+    (stroke (width 0) (type default) (color 0 0 0 0))
+  )
+  (polyline (pts (xy 198.12 134.62) (xy 198.12 135.89))
     (stroke (width 0) (type default) (color 0 0 0 0))
   )
@@
   (symbol (lib_id "power:GND") (at 82.55 25.4 0) (unit 1)
     (in_bom yes) (on_board yes) (fields_autoplaced)
-    (property "Reference" "#PWR?" (id 0) (at 82.55 31.75 0)
+    (property "Reference" "#PWR058" (id 0) (at 82.55 31.75 0)
       (effects (font (size 1.27 1.27)) hide)
     )
@@
   (symbol (lib_id "Connector:Conn_01x02_Male") (at 72.39 20.32 0) (unit 1)
     (in_bom yes) (on_board yes) (fields_autoplaced)
-    (property "Reference" "J?" (id 0) (at 73.025 15.24 0))
+    (property "Reference" "J8" (id 0) (at 73.025 15.24 0))
     (property "Value" "Conn_01x02_Male" (id 1) (at 73.025 17.78 0))
     (property "Footprint" "" (id 2) (at 72.39 20.32 0)
@@
   (symbol (lib_id "power:GND") (at 121.92 77.47 270) (unit 1)
     (in_bom yes) (on_board yes)
-    (property "Reference" "#PWR?" (id 0) (at 115.57 77.47 0)
+    (property "Reference" "#PWR059" (id 0) (at 115.57 77.47 0)
       (effects (font (size 1.27 1.27)) hide)
     )
@@
   (symbol (lib_id "Device:D_Schottky") (at 86.36 20.32 180) (unit 1)
     (in_bom yes) (on_board yes) (fields_autoplaced)
-    (property "Reference" "D?" (id 0) (at 86.6775 13.97 0))
+    (property "Reference" "D12" (id 0) (at 86.6775 13.97 0))
     (property "Value" "D_Schottky" (id 1) (at 86.6775 16.51 0))
     (property "Footprint" "" (id 2) (at 86.36 20.32 0)
@@
   (symbol (lib_id "Device:D_Schottky") (at 44.45 20.32 180) (unit 1)
     (in_bom yes) (on_board yes) (fields_autoplaced)
-    (property "Reference" "D?" (id 0) (at 44.7675 13.97 0))
+    (property "Reference" "D10" (id 0) (at 44.7675 13.97 0))
     (property "Value" "D_Schottky" (id 1) (at 44.7675 16.51 0))
     (property "Footprint" "" (id 2) (at 44.45 20.32 0)
@@
   (symbol (lib_id "Device:R_Small") (at 124.46 82.55 0) (unit 1)
     (in_bom yes) (on_board yes)
-    (property "Reference" "R?" (id 0) (at 129.54 82.55 90))
+    (property "Reference" "R28" (id 0) (at 129.54 82.55 90))
     (property "Value" "10K" (id 1) (at 127 82.55 90))
     (property "Footprint" "" (id 2) (at 124.46 82.55 0)
@@
   (symbol (lib_id "Device:D_Schottky") (at 50.8 148.59 180) (unit 1)
     (in_bom yes) (on_board yes) (fields_autoplaced)
-    (property "Reference" "D?" (id 0) (at 51.1175 142.24 0))
+    (property "Reference" "D11" (id 0) (at 51.1175 142.24 0))
     (property "Value" "D_Schottky" (id 1) (at 51.1175 144.78 0))
     (property "Footprint" "" (id 2) (at 50.8 148.59 0)

Commit message: Component_selection
Parts:
- removed D10, D11: D_Schottky, symbol Device:D_Schottky
- added D10: BAT54C, Package_TO_SOT_SMD:SOT-23, symbol Diode:BAT54C
- C29, C30, C31, C32, C35, C36, C37: footprint (none) -> Capacitor_SMD:C_0603_1608Metric
- C33, C34: footprint (none) -> Capacitor_SMD:C_0805_2012Metric
- D12: value D_Schottky -> CDBU0130-HF; footprint (none) -> CDBU0130-HF:DIOM1709X85N
- D8: footprint (none) -> LED_SMD:LED_0805_2012Metric
- J4: value Jack-DC -> DCJ250-10-A-K1-K; footprint (none) -> DCJ250-10-A_XX-X_REVA:GCT_DCJ250-10-A_XX-X_REVA
- J8: value Conn_01x02_Male -> PWR_PIN; footprint (none) -> Connector_PinHeader_2.54mm:PinHeader_1x02_P2.54mm_Vertical
- L2: footprint (none) -> Inductor_SMD:L_0603_1608Metric
- R13, R14, R15, R16, R17, R18: footprint (none) -> Resistor_SMD:R_0805_2012Metric
- R19, R20, R21, R22, R23, R28: footprint (none) -> Resistor_SMD:R_0603_1608Metric
- U5: footprint QFN50P400X400X100-25N -> BQ24195RGER:QFN50P400X400X100-25N
Connections:
- net VIN: now also D10.3
- net DC_JACK: now reaches J4.1
- net DC_JACK: now also D10.2
- net USB_VBUS: now reaches J5.1 (VBUS)
- net USB_VBUS: now also D10.1

Commit message: layout
Parts:
- removed D12: CDBU0130-HF, CDBU0130-HF:DIOM1709X85N, symbol Device:D_Schottky
- removed J8: PWR_PIN, Connector_PinHeader_2.54mm:PinHeader_1x02_P2.54mm_Vertical, symbol Connector:Conn_01x02_Male
- removed Q3, Q5: Si2312DS, Package_TO_SOT_SMD:SOT-23, symbol Transistor_FET:Si2319CDS
- added C39, C40: 1uF, Capacitor_SMD:C_0603_1608Metric, symbol Device:C_Small
- added IC1: BD33HC5MEFJ-ME2, BD33HC5MEFJ-ME2:SOIC127P600X100-8N, symbol BD33HC5MEFJ-ME2:BD33HC5MEFJ-ME2
- added Q1, Q3: Si2312DS, Package_TO_SOT_SMD:SOT-23, symbol Transistor_FET:BSN20
- added R1: 0R, Resistor_SMD:R_0603_1608Metric, symbol Device:R_Small
- BT1: footprint (none) -> Connector_PinHeader_2.54mm:PinHeader_1x02_P2.54mm_Vertical
- J5: value USB_B_Mini -> USB_B_Micro; footprint (none) -> Connector_USB:USB_Micro-B_Molex-105017-0001
Connections:
- net +3V3: now also C39.2, IC1.1 (VO), IC1.2 (FB/VO_S), R1.1
- net GND: now also C39.1, C40.1, IC1.3 (GND), Q1.2 (S), Q3.2 (S)
- net OTG: now also Q3.3 (D)
- net PMID: now also C40.2, IC1.5 (EN), IC1.8 (VCC)
- net at C29.2, Q4.3 (G), R18.1: now also Q1.3 (D)
- net at R15.2, R16.1: now also Q1.1 (G)
- net at R13.2, R14.1: now also Q3.1 (G)
- new net PWR_SIGNAL: R1.2
- no-connect marks 3 -> 6

Commit message: DRC
Parts:
- removed D10: BAT54C, Package_TO_SOT_SMD:SOT-23, symbol Diode:BAT54C
- removed D7: SP0502BAHT, Package_TO_SOT_SMD:SOT-23, symbol Power_Protection:SP0502BAHT
- removed J5: USB_B_Micro, Connector_USB:USB_Micro-B_Molex-105017-0001, symbol Connector:USB_B_Mini
- removed R1: 0R, Resistor_SMD:R_0603_1608Metric, symbol Device:R_Small
- added C41: 1uF, Capacitor_SMD:C_0805_2012Metric, symbol Device:C_Small
- added C42: 0.01uF, Capacitor_SMD:C_0603_1608Metric, symbol Device:C_Small
- added C43: 10uF, Capacitor_SMD:C_0603_1608Metric, symbol Device:C_Small
- added PS1: TAR5SB33_TE85L,F_, TAR5S33:SOT95P275X140-5N, symbol TAR5SB33_TE85L_F_:TAR5SB33_TE85L,F_
- added R2: 130R, Resistor_SMD:R_0805_2012Metric, symbol Device:R_Small
- J4: footprint DCJ250-10-A_XX-X_REVA:GCT_DCJ250-10-A_XX-X_REVA -> Connector_BarrelJack:BarrelJack_Horizontal
Connections:
- net DC_JACK is gone; now on net VIN: J4.1
- net GND: now also C41.1, C42.2, C43.1, PS1.2 (GND)
- net VIN: now also C41.2, PS1.1 (VIN), PS1.3 (CONTROL)
- new net: C42.1, PS1.4 (NOISE)
- new net: C43.2, PS1.5 (VOUT), R2.2
- new net Signal_VOUT: R2.1
- no-connect marks 6 -> 5
Other:
- moved on the sheet: BT1, C34, C35, C36, C37, C39, C40, IC1, L2

Commit message: ROUTE DONE
Parts:
- removed J4: DCJ250-10-A-K1-K, Connector_BarrelJack:BarrelJack_Horizontal, symbol Connector:Jack-DC
- added J4: USB4125-GF-A-0190_REVA2, USB4125-GF-A-0190_REVA2:GCT_USB4125-GF-A-0190_REVA2, symbol USB4125-GF-A-0190_REVA2:USB4125-GF-A-0190_REVA2
- added R31, R32: 5.1K, Resistor_SMD:R_0603_1608Metric, symbol Device:R_Small
- R23: value 100R -> 200R
Connections:
- net GND: now also J4.A12 (GND), J4.B12 (GND), J4.S1 (SHIELD), J4.S2 (SHIELD), J4.S3 (SHIELD), J4.S4 (SHIELD), R31.1, R32.1
- net VIN: now also J4.A9 (VBUS), J4.B9 (VBUS)
- net D+ renamed PMIC_D+
- net D- renamed PMIC_D-
- new net: J4.B5 (CC2), R31.2
- new net: J4.A5 (CC1), R32.2
