File: Hertz200/PCB_DESIGN/HERTZ200/MP2636.kicad_sch (KiCad schematic)
At the start: 53 parts, among them IC1 BD33HC5MEFJ-ME2, IC3 BQ29701DSET, J8 USB4125-GF-A-0190_REVA2, U5 CSD16406Q3, U6 MP2636GR-P, U9 CSD16406Q3

Commit message: BOM
Parts:
- removed R41: 10K, Resistor_SMD:R_0603_1608Metric, symbol Device:R_Small
- removed U5, U9: CSD16406Q3, CSD16406Q3:TRANS_CSD16406Q3, symbol CSD16406Q3:CSD16406Q3
- added Q1, Q3: CSD16301Q2, Package_SON:Texas_DQK, symbol Transistor_FET:CSD16301Q2
- C20, C48: value 1uF -> 0.1uF
- R14, R15: footprint Resistor_SMD:R_0603_1608Metric -> Resistor_SMD:R_0805_2012Metric
Connections:
- net GND: now also U6.26 (FREQ), Q1.4 (S), Q1.7 (S), Q3.4 (S), Q3.7 (S)
- net COUT: no longer names the net of IC3.2 (COUT), R15.2
- net COUT: now also Q3.3 (G)
- net DOUT: no longer names the net of IC3.3 (DOUT), R14.2
- net DOUT: now also Q1.3 (G)
- new net: Q1.1 (D), Q1.2 (D), Q1.5 (D), Q1.6 (D), Q1.8 (D), Q3.1 (D), Q3.2 (D), Q3.5 (D), Q3.6 (D), Q3.8 (D)
Other:
- moved on the sheet: R14, R15
