File: Hertz200/PCB_DESIGN/HERTZ200/SIM7020E.kicad_sch (KiCad schematic)
At the start: 35 parts, among them J1 SMA_CONNECTOR, J2 503960-0696, J5 105164-0001, Q2 BC847, U2 SIM7020E, U3 TXB0104PW, U7 100uF, U8 100uF

Commit message: ROUTE DONE
Parts:
- Q2: value BC847 -> BC847-T
Changed lines of the file:
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@@
       (effects (font (size 1.27 1.27)) (justify left))
     )
-    (property "Value" "BC847" (id 1) (at 64.77 171.4499 0)
+    (property "Value" "BC847-T" (id 1) (at 64.77 171.4499 0)
       (effects (font (size 1.27 1.27)) (justify left))
     )

Commit message: update
Parts:
- removed D6: ESD, Diode_SMD:D_0603_1608Metric, symbol ESD:ESD3V3D9-TP
Changed lines of the file:
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@@
   (junction (at 269.24 118.11) (diameter 0) (color 0 0 0 0)
   )
+  (junction (at 87.63 110.49) (diameter 0) (color 0 0 0 0)
+  )
   (junction (at 52.07 110.49) (diameter 0) (color 0 0 0 0)
   )
@@
   (junction (at 151.13 26.67) (diameter 0) (color 0 0 0 0)
   )
-  (junction (at 87.63 127) (diameter 0) (color 0 0 0 0)
-  )
   (junction (at 63.5 110.49) (diameter 0) (color 0 0 0 0)
   )
@@
   (junction (at 41.91 110.49) (diameter 0) (color 0 0 0 0)
   )
-  (junction (at 87.63 110.49) (diameter 0) (color 0 0 0 0)
-  )
   (junction (at 269.24 120.65) (diameter 0) (color 0 0 0 0)
   )
@@
   )
   (junction (at 237.49 40.64) (diameter 0) (color 0 0 0 0)
-  )
-  (junction (at 97.79 110.49) (diameter 0) (color 0 0 0 0)
   )
   (junction (at 90.17 185.42) (diameter 0) (color 0 0 0 0)
@@
     (stroke (width 1) (type default) (color 0 0 0 0))
   )
-  (wire (pts (xy 87.63 110.49) (xy 97.79 110.49))
-    (stroke (width 0) (type default) (color 0 0 0 0))
-  )
   (wire (pts (xy 88.9 163.83) (xy 88.9 162.56))
     (stroke (width 0) (type default) (color 0 0 0 0))
@@
     (stroke (width 0) (type default) (color 0 0 0 0))
   )
-  (wire (pts (xy 97.79 106.68) (xy 97.79 110.49))
-    (stroke (width 0) (type default) (color 0 0 0 0))
-  )
   (wire (pts (xy 204.47 138.43) (xy 204.47 140.97))
     (stroke (width 0) (type default) (color 0 0 0 0))
@@
   )
   (wire (pts (xy 229.87 100.33) (xy 226.06 100.33))
+    (stroke (width 0) (type default) (color 0 0 0 0))
+  )
+  (wire (pts (xy 87.63 107.95) (xy 87.63 110.49))
     (stroke (width 0) (type default) (color 0 0 0 0))
   )
@@
     (stroke (width 0) (type default) (color 0 0 0 0))
   )
-  (wire (pts (xy 97.79 110.49) (xy 97.79 111.76))
-    (stroke (width 0) (type default) (color 0 0 0 0))
-  )
   (wire (pts (xy 41.91 127) (xy 41.91 128.27))
     (stroke (width 0) (type default) (color 0 0 0 0))
@@
   )
   (wire (pts (xy 78.74 163.83) (xy 88.9 163.83))
-    (stroke (width 0) (type default) (color 0 0 0 0))
-  )
-  (wire (pts (xy 87.63 127) (xy 97.79 127))
     (stroke (width 0) (type default) (color 0 0 0 0))
   )
@@
     (pin "+")
     (pin "-")
-  )
-  (symbol (lib_id "ESD:ESD3V3D9-TP") (at 97.79 111.76 270) (unit 1)
-    (in_bom yes) (on_board yes)
-    (property "Reference" "D6" (id 0) (at 101.6 115.57 90)
-      (effects (font (size 1.27 1.27)) (justify left))
-    )
-    (property "Value" "ESD" (id 1) (at 101.6 119.38 90)
-      (effects (font (size 1.27 1.27)) (justify left))
-    )
-    (property "Footprint" "Diode_SMD:D_0603_1608Metric" (id 2) (at 101.6 121.92 0)
-      (effects (font (size 1.27 1.27)) (justify left) hide)
-    )
-    (property "Datasheet" "https://www.mouser.jp/datasheet/2/258/ESD3V3D9(SOD-923)-479119.pdf" (id 3) (at 99.06 121.92 0)
-      (effects (font (size 1.27 1.27)) (justify left) hide)
-    )
-    (property "Description" "ESD Suppressors / TVS Diodes Uni-dir 10mA, 3.3V" (id 4) (at 96.52 121.92 0)
-      (effects (font (size 1.27 1.27)) (justify left) hide)
-    )
-    (property "Height" "0.43" (id 5) (at 93.98 121.92 0)
-      (effects (font (size 1.27 1.27)) (justify left) hide)
-    )
-    (property "Manufacturer_Name" "Micro Commercial Components (MCC)" (id 6) (at 91.44 121.92 0)
-      (effects (font (size 1.27 1.27)) (justify left) hide)
-    )
-    (property "Manufacturer_Part_Number" "ESD3V3D9-TP" (id 7) (at 88.9 121.92 0)
-      (effects (font (size 1.27 1.27)) (justify left) hide)
-    )
-    (property "Mouser Part Number" "833-ESD3V3D9-TP" (id 8) (at 86.36 121.92 0)
-      (effects (font (size 1.27 1.27)) (justify left) hide)
-    )
-    (property "Mouser Price/Stock" "https://www.mouser.co.uk/ProductDetail/Micro-Commercial-Components-MCC/ESD3V3D9-TP?qs=WJd%252B7yD6my3RbvY7hgxwaQ%3D%3D" (id 9) (at 83.82 121.92 0)
-      (effects (font (size 1.27 1.27)) (justify left) hide)
-    )
-    (property "Arrow Part Number" "ESD3V3D9-TP" (id 10) (at 81.28 121.92 0)
-      (effects (font (size 1.27 1.27)) (justify left) hide)
-    )
-    (property "Arrow Price/Stock" "https://www.arrow.com/en/products/esd3v3d9-tp/micro-commercial-components" (id 11) (at 78.74 121.92 0)
-      (effects (font (size 1.27 1.27)) (justify left) hide)
-    )
-    (pin "1")
-    (pin "2")
   )
   (symbol (lib_id "power:GND") (at 139.7 76.2 0) (mirror y) (unit 1)
@@
     (pin "9")
   )
-  (symbol (lib_id "power:+3.3V") (at 97.79 106.68 0) (unit 1)
-    (in_bom yes) (on_board yes) (fields_autoplaced)
-    (property "Reference" "#PWR09" (id 0) (at 97.79 110.49 0)
-      (effects (font (size 1.27 1.27)) hide)
-    )
-    (property "Value" "+3.3V" (id 1) (at 97.79 101.6 0))
-    (property "Footprint" "" (id 2) (at 97.79 106.68 0)
-      (effects (font (size 1.27 1.27)) hide)
-    )
-    (property "Datasheet" "" (id 3) (at 97.79 106.68 0)
-      (effects (font (size 1.27 1.27)) hide)
-    )
+  (symbol (lib_id "power:+3.3V") (at 87.63 107.95 0) (unit 1)
+    (in_bom yes) (on_board yes) (fields_autoplaced)
+    (property "Reference" "#PWR09" (id 0) (at 87.63 111.76 0)
+      (effects (font (size 1.27 1.27)) hide)
+    )
+    (property "Value" "+3.3V" (id 1) (at 87.63 102.87 0))
+    (property "Footprint" "" (id 2) (at 87.63 107.95 0)
+      (effects (font (size 1.27 1.27)) hide)
+    )
+    (property "Datasheet" "" (id 3) (at 87.63 107.95 0)
+      (effects (font (size 1.27 1.27)) hide)
+    )
